Commit message: [done]7.15

File: src/bbot_demo/src/bbot_description/urdf/bbot.urdf.xacro (robot description, xacro)
@@ -3,3 +3,10 @@
   <xacro:include filename="bbot_description.xacro"/>
   <xacro:include filename="ros2_control.xacro"/>
+  <!-- <xacro:include filename="common_properties.xacro"/> -->
+  <xacro:include filename="arm.xacro"/>
+  <joint name="arm_base_joint" type="fixed">
+    <parent link="base_link"/>
+    <child link="arm_base_link"/>
+    <origin xyz="0.05 0 0.2" rpy="0 0 0"/>
+  </joint>
 </robot>

File: src/bbot_demo/src/bbot_description/urdf/ros2_control.xacro (robot description, xacro)
@@ -3,6 +3,10 @@
     <ros2_control name= "baseHardwareInterface" type= "system">
         <hardware>
-            <plugin>mock_components/GenericSystem</plugin>
-            <param name="calculate_dynamics" >true</param>
+            <!-- <plugin>mock_components/GenericSystem</plugin> -->
+            <!-- <param name="calculate_dynamics" >true</param> -->
+            <plugin>mobile_base_hardware/MobileBaseHardwareInterface</plugin>
+            <param name="left_motor_id">10</param>
+            <param name="right_motor_id">20</param>
+            <param name="dynamixel_port">/dev/ttyACM0</param>
         </hardware>
         <joint name="left_wheel_joint">
